Commit message: end effector to an XYZ

File: install/urdf_humble_test_moveit_config/share/urdf_humble_test_moveit_config/config/urdf_humble_test.ros2_control.xacro (robot description, xacro)
@@ -1 +1,54 @@
-/home/devika/robo_ws/src/urdf_humble_test_moveit_config/config/urdf_humble_test.ros2_control.xacro
+<?xml version="1.0"?>
+<robot xmlns:xacro="http://www.ros.org/wiki/xacro">
+    <xacro:macro name="urdf_humble_test_ros2_control" params="name initial_positions_file">
+        <xacro:property name="initial_positions" value="${load_yaml(initial_positions_file)['initial_positions']}"/>
+        <ros2_control name="${name}" type="system">
+            <hardware>
+                <!-- By default, set up controllers for simulation. This won't work on real hardware -->
+                <plugin>mock_components/GenericSystem</plugin>
+            </hardware>
+            <joint name="joint_1">
+                <command_interface name="position"/>
+                <state_interface name="position">
+                  <param name="initial_value">${initial_positions['joint_1']}</param>
+                </state_interface>
+                <state_interface name="velocity"/>
+            </joint>
+            <joint name="joint_2">
+                <command_interface name="position"/>
+                <state_interface name="position">
+                  <param name="initial_value">${initial_positions['joint_2']}</param>
+                </state_interface>
+                <state_interface name="velocity"/>
+            </joint>
+            <joint name="joint_3">
+                <command_interface name="position"/>
+                <state_interface name="position">
+                  <param name="initial_value">${initial_positions['joint_3']}</param>
+                </state_interface>
+                <state_interface name="velocity"/>
+            </joint>
+            <joint name="joint_4">
+                <command_interface name="position"/>
+                <state_interface name="position">
+                  <param name="initial_value">${initial_positions['joint_4']}</param>
+                </state_interface>
+                <state_interface name="velocity"/>
+            </joint>
+            <joint name="joint_5">
+                <command_interface name="position"/>
+                <state_interface name="position">
+                  <param name="initial_value">${initial_positions['joint_5']}</param>
+                </state_interface>
+                <state_interface name="velocity"/>
+            </joint>
+            <joint name="joint_6">
+                <command_interface name="position"/>
+                <state_interface name="position">
+                  <param name="initial_value">${initial_positions['joint_6']}</param>
+                </state_interface>
+                <state_interface name="velocity"/>
+            </joint>
+        </ros2_control>
+    </xacro:macro>
+</robot>

File: install/urdf_humble_test_moveit_config/share/urdf_humble_test_moveit_config/config/urdf_humble_test.urdf.xacro (robot description, xacro)
@@ -1 +1,9 @@
-/home/devika/robo_ws/src/urdf_humble_test_moveit_config/config/urdf_humble_test.urdf.xacro
+<?xml version="1.0"?>
+<robot xmlns:xacro="http://www.ros.org/wiki/xacro" name="urdf_humble_test">
+    <xacro:arg name="initial_positions_file" default="initial_positions.yaml" />
+    <!-- Import urdf_humble_test urdf file -->
+    <xacro:include filename="$(find urdf_humble_test)/urdf/model.urdf" />
+    <!-- Import control_xacro -->
+    <xacro:include filename="urdf_humble_test.ros2_control.xacro" />
+    <xacro:urdf_humble_test_ros2_control name="FakeSystem" initial_positions_file="$(arg initial_positions_file)"/>
+</robot>

File: src/urdf_humble_test/urdf/model.urdf (robot description, URDF)
Before this commit: robot urdf_humble_test, 9 links, 8 joints
Links:
- added link camera_link; visual box size=0.05 0.05 0.05
- added link camera_link_optical
Joints:
- added joint camera_joint: type fixed, parent link_5, child camera_link, origin xyz=-0.025 0.0 0.0 rpy=-1.57 3.14 1.57
- added joint camera_optical_joint: type fixed, parent camera_link, child camera_link_optical, origin xyz=0.0 0.0 0.0 rpy=-1.5708 0 -1.5708
- joint base_joint: origin xyz=0.0 0.0 0.0 rpy=0 0 0 -> xyz=0.0 0.0 -0.17 rpy=0 0 0
