Commit message: latest urdf

File: install/urdf_humble_test/share/urdf_humble_test/urdf/model.urdf (robot description, URDF)
Before this commit: robot urdf_humble_test, 11 links, 10 joints
Links:
- removed link camera_link
- removed link camera_link_optical
- added link link_8, mass 0.0657970930356421; collision mesh filename=package://urdf_humble_test/meshes/link_8.STL; visual mesh filename=package://urdf_humble_test/meshes/link_8.STL
- added link link_9, mass 0.0599258931002066; collision mesh filename=package://urdf_humble_test/meshes/link_9.STL; visual mesh filename=package://urdf_humble_test/meshes/link_9.STL
- link base_link: mass 0.605406509419497 -> 1.26158792714375
- link link_1: mass 0.77988040158824 -> 1.58252995063954
- link link_2: mass 0.443829266836424 -> 0.563584848829252
- link link_3: mass 1.67091128229235 -> 1.68158687764889
- link link_4: mass 0.186464706015941 -> 0.279984808714352
- link link_5: mass 0.383985526073569 -> 0.445153140088307
- link link_6: mass 0.0188998061392809 -> 0.0156031455954719
- link link_7: mass 0.0711438414703714 -> 0.0157543709875629
Joints:
- removed joint camera_joint
- removed joint camera_optical_joint
- added joint joint_8: type prismatic, parent link_5, child link_8, origin xyz=-0.0333725122311634 -0.114253153953276 -0.130847171307248 rpy=-3.14159265358979 1.28032965573961 3.14159265358979, axis 0 0 -1, limit lower=-0.042 upper=0 effort=0 velocity=0, mimic joint=joint_6 multiplier=-0.0042 offset=0
- added joint joint_9: type prismatic, parent link_5, child link_9, origin xyz=-0.0410222529877187 -0.136871142575247 -0.15643834277427 rpy=3.14159265358979 -1.28032965573961 0, axis 0 0 1, limit lower=-0.042 upper=0 effort=0 velocity=0, mimic joint=joint_6 multiplier=-0.0042 offset=0
- joint joint_1: axis 0 1 0 -> 0 0 1; limit lower=-3.1 upper=3.1 effort=0 velocity=0 -> lower=-3.14 upper=3.14 effort=0 velocity=0; origin xyz=-0.12173 -0.02365 0 rpy=1.5707963267949 0 0 -> xyz=0 0 0 rpy=0 0 0
- joint joint_2: axis 0 0 1 -> 0 0 -1; origin xyz=0 0.16104 -0.02365 rpy=0 0 0 -> xyz=-0.0589237850211093 -0.0176135617858798 0.196439999999998 rpy=1.5707963267949 0 1.86126299785025
- joint joint_3: axis 0 0 -1 -> 1 0 0; limit lower=0 upper=5.4 effort=0 velocity=0 -> lower=-6.28 upper=0 effort=0 velocity=0; origin xyz=0.38703 -0.10104 0 rpy=0 0 0 -> xyz=-0.349766547153894 0.0127813337346238 0 rpy=0 1.5707963267949 0
- joint joint_4: origin xyz=-0.38609 0.21104 0 rpy=0 0 0 -> xyz=0 0.120795067593268 0.44489274173121 rpy=0 1.5707963267949 0
- joint joint_5: axis 0.173285966010945 -0.984871552022726 0 -> -0.218564021615717 -0.646228246342021 -0.731176327628897; origin xyz=-0.0225 -0.02681 0.12075 rpy=0 0 -0.872490093071967 -> xyz=0.0475438829920029 0.0402600197471117 0.00549999999999323 rpy=0 1.28032965573954 0
- joint joint_6: axis 0 0 1 -> 0 0 -1; limit lower=0 upper=20 effort=0 velocity=0 -> lower=0 upper=10 effort=0 velocity=0; origin xyz=0.0154118344148917 -0.0875777161152765 -0.12075 rpy=0 0 1.74498018614393 -> xyz=-0.0333725122311634 -0.114253153953276 -0.130847171307248 rpy=-3.14159265358979 1.28032965573961 3.14159265358979
- joint joint_7: limit lower=0 upper=0.11 effort=0 velocity=0 -> lower=-10 upper=0 effort=0 velocity=0; mimic joint=joint_6 multiplier=0.005 offset=0 -> joint=joint_6 multiplier=-1 offset=0; origin xyz=0.0154118344148917 -0.0875777161152765 -0.12075 rpy=0 0 1.74498018614393 -> xyz=-0.0410222529877187 -0.136871142575247 -0.15643834277427 rpy=3.14159265358979 -1.28032965573961 0; type prismatic -> revolute

File: src/urdf_humble_test/urdf/model.urdf (robot description, URDF)
Before this commit: robot urdf_humble_test, 11 links, 10 joints
Links:
- removed link camera_link
- removed link camera_link_optical
- added link link_8, mass 0.0657970930356421; collision mesh filename=package://urdf_humble_test/meshes/link_8.STL; visual mesh filename=package://urdf_humble_test/meshes/link_8.STL
- added link link_9, mass 0.0599258931002066; collision mesh filename=package://urdf_humble_test/meshes/link_9.STL; visual mesh filename=package://urdf_humble_test/meshes/link_9.STL
- link base_link: mass 0.605406509419497 -> 1.26158792714375
- link link_1: mass 0.77988040158824 -> 1.58252995063954
- link link_2: mass 0.443829266836424 -> 0.563584848829252
- link link_3: mass 1.67091128229235 -> 1.68158687764889
- link link_4: mass 0.186464706015941 -> 0.279984808714352
- link link_5: mass 0.383985526073569 -> 0.445153140088307
- link link_6: mass 0.0188998061392809 -> 0.0156031455954719
- link link_7: mass 0.0711438414703714 -> 0.0157543709875629
Joints:
- removed joint camera_joint
- removed joint camera_optical_joint
- added joint joint_8: type prismatic, parent link_5, child link_8, origin xyz=-0.0333725122311634 -0.114253153953276 -0.130847171307248 rpy=-3.14159265358979 1.28032965573961 3.14159265358979, axis 0 0 -1, limit lower=-0.042 upper=0 effort=0 velocity=0, mimic joint=joint_6 multiplier=-0.0042 offset=0
- added joint joint_9: type prismatic, parent link_5, child link_9, origin xyz=-0.0410222529877187 -0.136871142575247 -0.15643834277427 rpy=3.14159265358979 -1.28032965573961 0, axis 0 0 1, limit lower=-0.042 upper=0 effort=0 velocity=0, mimic joint=joint_6 multiplier=-0.0042 offset=0
- joint joint_1: axis 0 1 0 -> 0 0 1; limit lower=-3.1 upper=3.1 effort=0 velocity=0 -> lower=-3.14 upper=3.14 effort=0 velocity=0; origin xyz=-0.12173 -0.02365 0 rpy=1.5707963267949 0 0 -> xyz=0 0 0 rpy=0 0 0
- joint joint_2: axis 0 0 1 -> 0 0 -1; origin xyz=0 0.16104 -0.02365 rpy=0 0 0 -> xyz=-0.0589237850211093 -0.0176135617858798 0.196439999999998 rpy=1.5707963267949 0 1.86126299785025
- joint joint_3: axis 0 0 -1 -> 1 0 0; limit lower=0 upper=5.4 effort=0 velocity=0 -> lower=-6.28 upper=0 effort=0 velocity=0; origin xyz=0.38703 -0.10104 0 rpy=0 0 0 -> xyz=-0.349766547153894 0.0127813337346238 0 rpy=0 1.5707963267949 0
- joint joint_4: origin xyz=-0.38609 0.21104 0 rpy=0 0 0 -> xyz=0 0.120795067593268 0.44489274173121 rpy=0 1.5707963267949 0
- joint joint_5: axis 0.173285966010945 -0.984871552022726 0 -> -0.218564021615717 -0.646228246342021 -0.731176327628897; origin xyz=-0.0225 -0.02681 0.12075 rpy=0 0 -0.872490093071967 -> xyz=0.0475438829920029 0.0402600197471117 0.00549999999999323 rpy=0 1.28032965573954 0
- joint joint_6: axis 0 0 1 -> 0 0 -1; limit lower=0 upper=20 effort=0 velocity=0 -> lower=0 upper=10 effort=0 velocity=0; origin xyz=0.0154118344148917 -0.0875777161152765 -0.12075 rpy=0 0 1.74498018614393 -> xyz=-0.0333725122311634 -0.114253153953276 -0.130847171307248 rpy=-3.14159265358979 1.28032965573961 3.14159265358979
- joint joint_7: limit lower=0 upper=0.11 effort=0 velocity=0 -> lower=-10 upper=0 effort=0 velocity=0; mimic joint=joint_6 multiplier=0.005 offset=0 -> joint=joint_6 multiplier=-1 offset=0; origin xyz=0.0154118344148917 -0.0875777161152765 -0.12075 rpy=0 0 1.74498018614393 -> xyz=-0.0410222529877187 -0.136871142575247 -0.15643834277427 rpy=3.14159265358979 -1.28032965573961 0; type prismatic -> revolute

Commit message: added camera and xyz poli

File: install/urdf_humble_test/share/urdf_humble_test/urdf/model.urdf (robot description, URDF)
Before this commit: robot urdf_humble_test, 11 links, 10 joints
Links:
- added link camera_link_optical
Joints:
- added joint camera_optical_joint: type fixed, parent link_6, child camera_link_optical, origin xyz=0.04 0.05 0.0 rpy=0 0 -0.785

Commit message: camera crct orientation

File: install/urdf_humble_test/share/urdf_humble_test/urdf/model.urdf (robot description, URDF)
Before this commit: robot urdf_humble_test, 12 links, 11 joints
Links:
- added link camera_link
Joints:
- added joint camera_joint: type fixed, parent link_6, child camera_link, origin xyz=0.04 0.05 0.0 rpy=-1.57 0 -0.785
- joint camera_optical_joint: origin xyz=0.04 0.05 0.0 rpy=0 0 -0.785 -> xyz=0 0 0 rpy=-1.5708 0 -1.5708; parent link_6 -> camera_link

Commit message: added fake joints

File: install/urdf_humble_test/share/urdf_humble_test/urdf/model.urdf (robot description, URDF)
Before this commit: robot urdf_humble_test, 13 links, 12 joints
Links:
- added link fake_link
Joints:
- added joint fake_joint: type revolute, parent link_5, child fake_link, origin xyz=0 0 0 rpy=0 0 0, axis 0 0 1, limit lower=-3.14159 upper=3.14159 effort=0 velocity=0

Commit message: added fake joint in controllers too now orientation seems to be working too

File: install/urdf_humble_test/share/urdf_humble_test/urdf/model.urdf (robot description, URDF)
Before this commit: robot urdf_humble_test, 14 links, 13 joints
Links:
- link fake_link: mass None -> 0.001

Commit message: a lot of changes, actually, i lost track of it

File: install/urdf_humble_test/share/urdf_humble_test/urdf/model.urdf (robot description, URDF)
Before this commit: robot urdf_humble_test, 14 links, 13 joints
Joints:
- joint fake_joint: origin xyz=0 0 0 rpy=0 0 0 -> xyz=-0.06 -0.175 -0.2 rpy=-0.3 2.355 1.37
- joint joint_4: limit lower=-3.14 upper=3.14 effort=0 velocity=0 -> lower=-1.0 upper=1.14 effort=0 velocity=0
- joint joint_6: limit lower=0 upper=10 effort=0 velocity=0 -> lower=0 upper=10 effort=10 velocity=0
- joint joint_7: limit lower=-10 upper=0 effort=0 velocity=0 -> lower=-10 upper=0 effort=5 velocity=0
- joint joint_8: limit lower=-0.042 upper=0 effort=0 velocity=0 -> lower=-0.042 upper=0 effort=10 velocity=0
- joint joint_9: limit lower=-0.042 upper=0 effort=0 velocity=0 -> lower=-0.042 upper=0 effort=10 velocity=0

Commit message: saving

File: install/urdf_humble_test/share/urdf_humble_test/urdf/model.urdf (robot description, URDF)
Before this commit: robot urdf_humble_test, 14 links, 13 joints
Links:
- link fake_link: geometry collision box size=0.005 0.005 0.005; visual box size=0.005 0.005 0.005
Joints:
- joint fake_joint: limit lower=-3.14159 upper=3.14159 effort=0 velocity=0 -> lower=-1.14159 upper=1.14159 effort=0 velocity=0
- joint joint_4: limit lower=-1.0 upper=1.14 effort=0 velocity=0 -> lower=-3.140 upper=3.14 effort=0 velocity=0
